Commit message: Created the joint state publisher with the TF frames

File: urdf/puzzlebot.urdf (robot description, URDF)
Before this commit: robot PuzzleBot, 4 links, 3 joints
Joints:
- joint wheel_coupler_joint: axis (none) -> 0 1 0; origin xyz=-0.08 -0.05 0 rpy=0 0 0 -> xyz=0 0 0 rpy=0 0 0; type fixed -> continuous
- joint wheel_coupler_joint_2: axis (none) -> 0 1 0; origin xyz=0.08 -0.05 0 rpy=0 0 0 -> xyz=0 0 0 rpy=0 0 0; type fixed -> continuous
