Commit message: Fixed launchfile error and rviz error with the puzzlebot model

File: urdf/puzzlebot_jetson_ed_urdf.urdf (robot description, URDF)
Before this commit: robot Puzzlebot Jetson-Lidar Ed., 2 links, 1 joints
Links:
- link chassis: geometry collision mesh filename=package://puzzlebot_challenge/models/MCR2_1000_13_Chassis.s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; visual mesh filename=package://puzzlebot_challenge/models/MCR2_1000_13_Chassis.s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

Commit message: Completed launch file and adjusted file directories

File: urdf/puzzlebot_jetson_ed_urdf.urdf (robot description, URDF)
Before this commit: robot PuzzleBot, 4 links, 3 joints
Links:
- link chassis: geometry collision mesh filename=package://puzzlebot_challenge/models/MCR2_1000_13_Chassis.s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; visual mesh filename=package://puzzlebot_challenge/models/MCR2_1000_13_Chassis.s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
- link wheel_coupler: geometry visual mesh filename=package://puzzlebot_challenge/models/MCR2_1000_1_1_Wheel_Co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
- link wheel_coupler_2: geometry visual mesh filename=package://puzzlebot_challenge/models/MCR2_1000_1_1_Wheel_Co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
