Commit message: update

File: localisation/urdf/puzzlebot_jetson_ed_urdf.urdf (robot description, URDF)
Before this commit: robot PuzzleBot, 4 links, 3 joints
Joints:
- joint wheel_coupler_joint: axis 0 1 0 -> (none); type continuous -> fixed
- joint wheel_coupler_joint_2: axis 0 1 0 -> (none); type continuous -> fixed
