Commit message: update

File: puzzlebot_challenge/urdf/puzzlebot.urdf (robot description, URDF)
Before this commit: robot PuzzleBot, 4 links, 3 joints
Links:
- added link nueva_pieza; collision mesh filename=package://puzzlebot_challenge/models/MCR2_1000_13_Chassis.s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; visual mesh filename=package://puzzlebot_challenge/models/MCR2_1000_13_Chassis.s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
Joints:
- added joint nueva_pieza_joint: type fixed, parent base_link, child nueva_pieza, origin xyz=1 0 0 rpy=0 0 0

Commit message: update

File: puzzlebot_challenge/urdf/puzzlebot.urdf (robot description, URDF)
Before this commit: robot PuzzleBot, 5 links, 4 joints
Links:
- removed link nueva_pieza
Joints:
- removed joint nueva_pieza_joint
